File: Hardware/ESP32_Thing_Plus.sch (EAGLE design)
At the start: 72 parts, among them Q1 2.5A/30V, Q2 MBT3904DW1T1, U1 MCP73831, U2 ESP3212, U3 AP2112K-3.3V, U4 FT231XS, U5 W25Q32FVSS, Y1 26MHz, Y2 32.768kHz

Commit message: Initial changes to board design
Parts:
- removed C17, C20, C21, C23, C25: 0.1uF, SparkFun-Capacitors:0.1UF-0603-25V-(+80/-20%)
- removed C18: 100pF, SparkFun-Capacitors:100PF-0603-50V-5%
- removed C22: 10uF, SparkFun-Capacitors:10UF-0603-6.3V-20%
- removed C24: 1.0uF, SparkFun-Capacitors:1.0UF-0603-16V-10%
- removed C26, C9: 15pF, SparkFun-Capacitors:15PF-0603-50V-5%
- removed C27: 3.0nF, esp32-thing-temp:3.0NF-0603-50V-5%
- removed C4: 10pF, SparkFun-Capacitors:10PF-0603-50V-5%
- removed C5: 10nF, SparkFun-Capacitors:10NF-0603-50V-10%
- removed C8: 5.6pF, esp32-thing-temp:5.6PF-50V-5%(0603)
- removed E1: ANTENNA, esp32-thing-temp:ANTENNATRACE-TUNED
- removed L1, L2: DNP, SparkFun-Passives:INDUCTOR0603
- removed R1: 10k, SparkFun-Resistors:10KOHM-1/10W-1%(0603)0603
- removed SJ3: JUMPER-PAD-3-2OF3_NC_BY_TRACE_SMALL, SparkFun-Passives:JUMPER-PAD-3-2OF3_NC_BY_TRACE_SMALL
- removed U5: W25Q32FVSS, SparkFun-DigitalIC:W25Q32FVSS
- removed Y1: 26MHz, things:CRYSTAL-GROUNDED3.2X2.5
- removed Y2: 32.768kHz, SparkFun-Clocks:CRYSTAL-32.768KHZSMD-3.2X1.5
- added J3: (no value), SparkFun-Connectors:QWIIC_CONNECTORJS-1MM
- added R10: 10k, SparkFun-Resistors:10KOHM-0603-1/10W-1%
- C1: value 270pF -> 0.1uF; device esp32-thing-temp:270PF-50V-5%(0603) -> SparkFun-Capacitors:0.1UF-0603-25V-5%
- C2: value 270pF -> 10uF; device esp32-thing-temp:270PF-50V-5%(0603) -> SparkFun-Capacitors:10UF-0805-10V-10%
- C3: value 10pF -> 0.1uF; device SparkFun-Capacitors:10PF-0603-50V-5% -> SparkFun-Capacitors:0.1UF-0603-25V-5%
- F1: value 500mA -> 6V/0.75A; device SparkFun-PowerIC:PTCSMD -> SparkFun-Fuses:PPTC_THREE-QUARTER-AMP
- LOGO1: value SFE_LOGO_NAME.2_INCH -> SFE_LOGO_NAME.1_INCH; device SparkFun-Aesthetics:SFE_LOGO_NAME.2_INCH -> SparkFun-Aesthetics:SFE_LOGO_NAME.1_INCH
- R2: value 20k -> 10k; device SparkFun-Resistors:20KOHM-0603-1/10W-1% -> SparkFun-Resistors:10KOHM-0603-1/10W-1%
- U2: value ESP3212 -> ESP-WROOM-32; device esp32-thing-temp:ESP3212 -> SparkFun-RF:ESP-WROOM-32
Connections:
- removed net 32K_XN: C26.2, J1.15, U2.32K_XN(GPIO33/ADC1:5/TOUCH8/RTC8), Y2.2
- removed net 32K_XP: C9.2, J1.16, U2.32K_XP(GPIO32/ADC1:4/TOUCH9/RTC9), Y2.1
- removed net 36: C1.2, J1.20, U2.SENSOR_VP(GPI36/ADC1:0/RTC0)
- removed net 37: C1.1, J1.19, U2.SENSOR_CAPP(GPI37/ADC1:1/RTC1)
- removed net 38: C2.1, J1.18, U2.SENSOR_CAPN(GPI38/ADC1:2/RTC2)
- removed net 39: C2.2, J1.17, U2.SENSOR_VN(GPI39/ADC1:3/RTC3)
- removed net CAP_10N: C27.1, C5.2, R2.2, U2.CAP1
- removed net FLASH_SCK: U2.(GPIO6/SPICLK/HS1_CLK/U1CTS)SD_CLK, U5.SCK
- removed net FLASH_SCS: U2.(GPIO11/SPICSO/HS1_CMD/U1RTS)SD_CMD, U5.!CS!
- removed net FLASH_SDI: U2.(GPIO8/SPID/HS1_DATA1)SD_DATA1, U5.SI(D0)
- removed net FLASH_SDO: U2.(GPIO7/SPI1/HS1_DATA0)SD_DATA0, U5.SO(D1)
- removed net FLASH_SHD: U2.(GPIO9/SPIHD/HS1_DATA2/U1RX)SD_DATA2, U5.!HOLD!(D3)
- removed net FLASH_SWP: U2.(GPIO10/SPIWP/HS1_DATA3/U1TX)SD_DATA3, U5.!WP!(D2)
- removed net FLASH_VDD: C24.1, SJ3.1, U2.VDD3P3_SDIO
- removed net LNA_IN: C8.1, L1.1, U2.LNA_IN
- removed net N$11: C17.1, SJ3.2, U5.VCC
- removed net N$13: C3.2, U2.XTAL_P, Y1.1
- removed net N$15: C4.2, U2.XTAL_N, Y1.2
- removed net N$4: C27.2, R2.1, U2.CAP2
- removed net TRACE_ANT: C8.2, E1.SIGNAL, L2.1
- new net 20: J2.14, U2.IO20
- new net 32: J1.18, U2.IO32
- new net 33: J1.17, U2.IO33
- net 0: now also J2.7, U2.IO0; no longer J2.9, U2.(ADC2:1/TOUCH1/RTC11/CLK_OUT1)GPIO0
- net 12: now also J1.12, R10.2, U2.IO12; no longer J1.8, U2.(GPIO12/ADC2:5/TOUCH5/RTC15/SPIQ)MTDI
- net 13: now also J1.11, U2.IO13; no longer J1.7, U2.(GPIO13/ADC2:4/TOUCH4/RTC14/SPID/U0CTS)MTCK
- net 14: now also J1.13, U2.IO14; no longer J1.9, U2.(GPIO14/ADC2:6/TOUCH6/RTC16/SPICLK)MTMS
- net 15: now also J1.10, U2.IO15; no longer J2.11, U2.(GPIO15/ADC2:3/TOUCH3/RTC13/SPICSO/U0RTS)MTDO
- net 16: now also J2.9, U2.IO16; no longer J2.6, U2.(HS1_DATA4)GPIO16
- net 17: now also J2.10, U2.IO17; no longer J2.7, U2.(HS1_DATA5)GPIO17
- net 18: now also J2.12, U2.IO18; no longer J2.13, U2.(VSPICLK/HS1_DATA7)GPIO18
- net 19: now also J2.13, U2.IO19; no longer J2.15, U2.(VSPIQ/HS2_DATA2)GPIO19
- net 2: now also J2.6, U2.IO2; no longer J2.10, U2.(ADC2:2/TOUCH2/RTC12/SPIWP)GPIO2
- net 21: now also J2.15, J3.3, U2.IO21; no longer J2.19, U2.(VSPIHD/HS2_CMD)GPIO21
- net 22: now also J2.18, J3.4, U2.IO22; no longer J2.16, U2.(VSPIWP/HS2_CLK)GPIO22
- net 23: now also J2.19, U2.IO23; no longer J2.14, U2.GPIO23
- net 25: now also J1.16, U2.IO25; no longer J1.12, U2.(DAC1/ADC2:8/RTC6)GPIO25
- net 26: now also J1.15, U2.IO26; no longer J1.11, U2.(DAC2/ADC2:9/RTC7)GPIO26
- net 27: now also J1.14, U2.IO27; no longer J1.10, U2.(ADC2:7/TOUCH7/RTC17)GPIO27
- net 3.3V: now also C1.1, C2.1, J3.2, R2.2, U2.3V3; no longer C18.1, C20.1, C21.1, C22.1, C23.1, C25.1, R1.2, SJ3.3, U2.VDD3P3_CPU, U2.VDD3P3_RTC, U2.VDDA, U2.VDDA3P3
- net 34: now also J1.20, U2.IO34; no longer J1.14, U2.VDET_1(GPI34/ADC1:6)
- net 35: now also J1.19, U2.IO35; no longer J1.13, U2.VDET_2(GPI35/ADC1:7)
- net 4: now also U2.IO4; no longer U2.(ADC2:0/TOUCH0/RTC10/SPIHD)GPIO4
- net 5: now also J2.11, U2.IO5; no longer J2.12, U2.(VSPICS0/HS1_DATA6)GPIO5
- net CHIP_PU: now also C3.1, R2.1, U2.EN; no longer R1.1, U2.CHIP_PU
- net GND: now also C1.2, C2.2, C3.2, J1.7, J1.8, J1.9, J3.1, R10.1, U2.GND@1, U2.GND@15, U2.GND@38; no longer C17.2, C18.2, C20.2, C21.2, C22.2, C23.2, C24.2, C25.2, C26.1, C3.1, C4.1, C5.1, C9.1, E1.GND, L1.2, L2.2, U5.GND, Y1.GND
- net U0RXD: now also J2.16, U2.RXD; no longer J2.17, U2.(GPIO3/CLK_OUT2/HS2_DATA0)U0RXD
- net U0TXD: now also J2.17, U2.TXD; no longer J2.18, U2.(GPIO1/CLK_OUT3/HS2_DATA1)U0TXD
Other:
- note removed: "32.768kHz RTC Crystal"
- note removed: "CHIP_PU is the ESP32's enable/reset pin. It must be pulled high to turn the ESP32 on."
- note removed: "ESP32 VCC Range: 2.8-3.6V"
- note removed: "Near VDDA 46, 43"
- note removed: "Near VDDA3P3 3, 4"
- note removed: "Near VDDA_LNA 1"
- note removed: "Near VDDPST_CPU 37"
- note removed: "Near VDDPST_RTC 19"
- note removed: "Near VDDPST_SDIO 26"
- note removed: "SJ3 allows selection between FLASH_VDD and 3.3V as the voltage supply to the flash IC."
- note removed: "W25Q32FVSS - 4MB SPI Flash"
- moved on the sheet: C1, C2, C3, R2

Commit message: Ready for qc review
Parts:
- added FD3, FD4: FIDUCIALUFIDUCIAL, SparkFun-Aesthetics:FIDUCIALUFIDUCIAL
Other:
- note added: "01"
- note added: "Original ESP32 Thing by Jim Lindblom ESP32 Thing Plus by Mike Hord"
- note added: "QWIIC Connector"
- note removed: "Jim Lindblom"
- note removed: "v10"
- moved on the sheet: C1, C2, C3, J3, R10, R2, U2

Commit message: Revised per QC double check
Other:
- note added: "Mike Hord"
- note added: "Original ESP32 Thing by Jim Lindblom"
- note removed: "Original ESP32 Thing by Jim Lindblom ESP32 Thing Plus by Mike Hord"
Changed lines of the file:
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@@
 <text x="332.74" y="104.14" size="2.54" layer="94" align="top-left">Headers</text>
 <text x="421.64" y="10.16" size="2.54" layer="94" align="top-left">01</text>
-<text x="355.6" y="8.89" size="1.27" layer="94" rot="MR180" align="top-left">Original ESP32 Thing by Jim Lindblom
-ESP32 Thing Plus by Mike Hord</text>
+<text x="273.812" y="0.762" size="1.778" layer="94" rot="MR180" align="top-left">Original ESP32 Thing by Jim Lindblom</text>
 <text x="93.98" y="231.14" size="2.032" layer="97" font="vector">SJ2 disconnects the
 power LED (for
@@
 <text x="381" y="114.3" size="1.778" layer="97" font="vector" align="top-center">If DTR is LOW, toggling RTS from HIGH to LOW resets to run mode.
 If RTS is HIGH, toggling DTR from LOW to HIGH resets to bootloader.</text>
-<text x="264.16" y="187.96" size="2.54" layer="91">QWIIC Connector</text>
+<text x="264.16" y="187.96" size="2.54" layer="94">QWIIC Connector</text>
 <wire x1="259.08" y1="99.06" x2="259.08" y2="193.04" width="0.1524" layer="97" style="longdash"/>
+<text x="358.14" y="7.62" size="3.81" layer="91">Mike Hord</text>
 </plain>
 <instances>
@@
 <instance part="GND14" gate="1" x="43.18" y="223.52"/>
 <instance part="U1" gate="G$1" x="208.28" y="248.92" rot="MR0"/>
-<instance part="GND9" gate="1" x="195.58" y="231.14" rot="MR0"/>
+<instance part="GND9" gate="1" x="195.58" y="218.44" rot="MR0"/>
 <instance part="GND11" gate="1" x="185.42" y="218.44" rot="MR0"/>
 <instance part="GND12" gate="1" x="175.26" y="238.76" smashed="yes" rot="MR0">
@@
 <instance part="R6" gate="G$1" x="185.42" y="228.6" rot="MR90"/>
 <instance part="R5" gate="G$1" x="190.5" y="241.3" rot="MR90"/>
-<instance part="GND10" gate="1" x="190.5" y="231.14" rot="MR0"/>
+<instance part="GND10" gate="1" x="190.5" y="218.44" rot="MR0"/>
 <instance part="SJ1" gate="G$1" x="185.42" y="241.3" smashed="yes" rot="R90">
 <attribute name="NAME" x="182.88" y="238.76" size="1.778" layer="95" rot="R90"/>
@@
 <instance part="R8" gate="G$1" x="226.06" y="27.94" rot="R90"/>
 <instance part="GND37" gate="1" x="226.06" y="17.78"/>
-<instance part="LOGO2" gate="G$1" x="12.7" y="10.16"/>
+<instance part="LOGO2" gate="G$1" x="244.856" y="11.176"/>
 <instance part="FD1" gate="G$1" x="429.26" y="27.94"/>
 <instance part="FD2" gate="G$1" x="426.72" y="25.4"/>
@@
 <wire x1="198.12" y1="246.38" x2="195.58" y2="246.38" width="0.1524" layer="91"/>
 <pinref part="GND9" gate="1" pin="GND"/>
-<wire x1="195.58" y1="246.38" x2="195.58" y2="233.68" width="0.1524" layer="91"/>
+<wire x1="195.58" y1="246.38" x2="195.58" y2="220.98" width="0.1524" layer="91"/>
 </segment>
 <segment>
@@
 <pinref part="R5" gate="G$1" pin="1"/>
 <pinref part="GND10" gate="1" pin="GND"/>
-<wire x1="190.5" y1="233.68" x2="190.5" y2="236.22" width="0.1524" layer="91"/>
-</segment>
-<segment>
+<wire x1="190.5" y1="220.98" x2="190.5" y2="236.22" width="0.1524" layer="91"/>
+</segment>
+<segment>

Commit message: Replaced EOL 1.0uF cap with newer one
Parts:
- C7: device SparkFun-Capacitors:1.0UF-0805-25V-(+80/-20%) -> SparkFun-Capacitors:1.0UF-0603-16V-10%-X7R
Changed lines of the file:
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@@
 <part name="C15" library="SparkFun-Capacitors" deviceset="4.7UF-6.3V-10%(0603)" device="0603" value="4.7uF"/>
 <part name="GND15" library="SparkFun-Aesthetics" deviceset="GND" device=""/>
-<part name="C7" library="SparkFun-Capacitors" deviceset="1.0UF" device="-0805-25V-(+80/-20%)" value="1.0uF"/>
+<part name="C7" library="SparkFun-Capacitors" deviceset="1.0UF" device="-0603-16V-10%-X7R" value="1.0uF"/>
 <part name="C10" library="SparkFun-Capacitors" deviceset="2.2UF" device="-0603-10V-20%" value="2.2uF"/>
 <part name="GND21" library="SparkFun-Aesthetics" deviceset="GND" device=""/>

Commit message: Feedback from review
Parts:
- removed C11, C14, C16: 0.1uF, SparkFun-Capacitors:0.1UF-0603-25V-(+80/-20%)
- removed C12, C13: 47pF, SparkFun-Capacitors:47PF-0603-50V-5%
- removed C15: 4.7uF, SparkFun-Capacitors:4.7UF-6.3V-10%(0603)0603
- removed C2: 10uF, SparkFun-Capacitors:10UF-0805-10V-10%
- removed C3: 0.1uF, SparkFun-Capacitors:0.1UF-0603-25V-5%
- removed D4: BLUE, SparkFun-LED:LED-BLUE0603
- removed F1: 6V/0.75A, SparkFun-Fuses:PPTC_THREE-QUARTER-AMP
- removed JP15: (no value), SparkFun-Connectors:USB_MICROB_PLUGCONN-11752
- removed R10: 10k, SparkFun-Resistors:10KOHM-0603-1/10W-1%
- removed R13, R14: 27, SparkFun-Resistors:27OHM1/10W1%(0603)0603-RES
- removed S2: BTN-0, SparkFun-Electromechanical:SWITCH-MOMENTARY-2SMD-4.6X2.8MM
- removed SJ1, SJ2: JUMPER-PAD-2-NC_BY_TRACE, SparkFun-Passives:JUMPER-PAD-2-NC_BY_TRACE
- added J4: (no value), SparkFun-Connectors:CONN_161X16_NO_SILK
- added LOGO4: FOUR_LAYER_WARNING, SparkFun-Aesthetics:FOUR_LAYER_WARNING
- added R1: 1k, SparkFun-Resistors:1KOHM-0603-1/10W-1%
- C1: value 0.1uF -> 10uF; device SparkFun-Capacitors:0.1UF-0603-25V-5% -> SparkFun-Capacitors:10UF-0603-6.3V-20%
- C10: value 2.2uF -> 1.0uF; device SparkFun-Capacitors:2.2UF-0603-10V-20% -> SparkFun-Capacitors:1.0UF-0402-16V-10%
- D3: value RED -> BLUE; device SparkFun-LED:LED-RED0603 -> SparkFun-LED:LED-BLUE0603
- J1: value (none) -> AMP FCI 10103594-0001LF; device SparkFun-Connectors:M20NOSILK -> SparkFun-Connectors:USB_MICRO-B_HALF_PTH
- J2: device SparkFun-Connectors:M20NOSILK -> SparkFun-Connectors:CONN_12NO_SILK
- JP2: device SparkFun-Connectors:M02JST-PTH-2 -> SparkFun-Connectors:CONN_02-JST-2MM-SMT
- LOGO1: value SFE_LOGO_NAME.1_INCH -> SFE_LOGO_FLAME.1_INCH; device SparkFun-Aesthetics:SFE_LOGO_NAME.1_INCH -> SparkFun-Aesthetics:SFE_LOGO_FLAME.1_INCH
- LOGO3: value SFE_LOGO_NAME.2_INCH -> SFE_LOGO_NAME_FLAME.1_INCH; device SparkFun-Aesthetics:SFE_LOGO_NAME.2_INCH -> SparkFun-Aesthetics:SFE_LOGO_NAME_FLAME.1_INCH
- R4: value 1K -> 1k; device SparkFun-Resistors:1KOHM-1/10W-1%(0603) -> SparkFun-Resistors:1KOHM-0603-1/10W-1%
- R5: value DNP -> 100K; device SparkFun-Passives:RESISTORPTH-1/6W -> SparkFun-Resistors:100KOHM-0402-1/16W-1%
- R8: value 330 -> 100K; device SparkFun-Resistors:330OHM1/10W1%(0603) -> SparkFun-Resistors:100KOHM-0402-1/16W-1%
- R9: value 10k -> 100K; device SparkFun-Resistors:10KOHM-1/10W-1%(0603)0603 -> SparkFun-Resistors:100KOHM-0402-1/16W-1%
- S1: device SparkFun-Electromechanical:SWITCH-MOMENTARY-2SMD-4.6X2.8MM -> SparkFun-Switches:MOMENTARY-SWITCH-SPST-2-SMD-4.6X2.8MM
- U2: value ESP-WROOM-32 -> ESP-WROOM-32NARROW; device SparkFun-RF:ESP-WROOM-32 -> SparkFun-RF:ESP-WROOM-32NARROW
- U4: value FT231XS -> CP2102N; device SparkFun-DigitalIC:FT231XS -> SparkFun-IC-Comms:CP2102N
Connections:
- net N$9 renamed CHG
- removed net 18: J2.12, U2.IO18
- removed net 19: J2.13, U2.IO19
- removed net 21: J2.15, J3.3, U2.IO21
- removed net 22: J2.18, J3.4, U2.IO22
- removed net 25: J1.16, U2.IO25
- removed net 26: J1.15, U2.IO26
- removed net 3.3V_F: C16.1, U4.!RESET, U4.3V3OUT, U4.VCCIO
- removed net 34: J1.20, U2.IO34
- removed net 4: J2.8, U2.IO4
- removed net 5: D4.A, J2.11, U2.IO5
- removed net N$16: R6.2, SJ1.1
- removed net N$3: R4.1, SJ2.1
- removed net N$7: R13.2, U4.USBDM
- removed net N$8: R14.2, U4.USBDP
- removed net SHIELD: JP15.SHIELD
- removed net U0RXD: J2.16, U2.RXD, U4.TXD
- removed net U0TXD: J2.17, U2.TXD, U4.RXD
- removed net VUSB-RAW: C11.1, F1.1, J1.2, J2.2, JP15.VCC
- new net A0: J4.5, U2.IO26
- new net A1: J4.6, U2.IO25
- new net A2: J4.7, U2.IO34
- new net A3: J4.8, U2.SENSOR_VN
- new net A4: J4.9, U2.SENSOR_VP
- new net A5: J4.10, U2.IO4
- new net EN: J2.2, R8.2, U3.EN
- new net MISO: J4.13, U2.IO19
- new net MOSI: J4.12, U2.IO18
- new net RX: U2.TXD, U4.RXD
- new net SCK: J4.11, U2.IO5
- new net SCL: J2.11, J3.4, U2.IO22
- new net SDA: J2.12, J3.3, U2.IO21
- new net TX: U2.RXD, U4.TXD
- new net VDD: U4.VDD
- net 0: no longer J2.7, R9.1, S2.2
- net 12: no longer J1.12, R10.2
- net 13: now also J2.4, R4.1; no longer J1.11
- net 14: now also J2.10; no longer J1.13
- net 15: now also J2.8; no longer J1.10
- net 16: now also J4.14; no longer J2.9
- net 17: now also J4.15; no longer J2.10
- net 2: no longer J2.6
- net 20: now also J2.5; no longer J2.14
- net 23: now also J4.16; no longer J2.19
- net 27: now also J2.6; no longer J1.14
- net 3.3V: now also J4.2, R1.1, U4.VIO; no longer C2.1, J1.5, J2.5, R9.2, SJ2.2
- net 32: now also J2.9; no longer J1.18
- net 33: now also J2.7; no longer J1.17
- net 35: now also R5.1, R9.2; no longer J1.19
- net CHIP_PU: now also J4.1, S1.4; no longer C3.1, J1.6, S1.2
- net D+: now also J1.D+, U4.D+; no longer C13.1, JP15.D+, R14.1
- net D-: now also J1.D-, U4.D-; no longer C12.1, JP15.D-, R13.1
- net DTR: now also U4.DTR; no longer U4.!DTR
- net GND: now also J1.GND, J4.4, R9.1, U4.GND; no longer C11.2, C12.2, C13.2, C14.2, C15.2, C16.2, C2.2, C3.2, J1.1, J1.4, J1.7, J1.8, J1.9, J2.1, J2.20, J2.4, JP15.GND, R10.1, R5.1, R8.1, S2.1, U4.GND@16, U4.GND@6
- net N$1: now also R1.2, U4.!RSTB; no longer D4.C, R8.2
- net N$14: now also R6.2; no longer R5.2, SJ1.2
- net RTS: now also U4.RTS; no longer U4.!RTS
- net VIN: now also R8.1; no longer U3.EN
- net V_BATT: now also J2.1, R5.2; no longer J1.3, J2.3
- net V_USB: now also J1.VBUS, J2.3, U4.VREGIN; no longer C14.1, C15.1, F1.2, U4.VCC
Other:
- note added: "CP2102N (USB-to-Serial Converter)"
- note removed: "FT231XS (USB-to-Serial Converter)"
- note removed: "GPIO0 Button"
- note removed: "GPIO5 LED"
- note removed: "SJ2 disconnects the power LED (for power saving)."
- moved on the sheet: C1, C10, C7, D2, D3, Q1, R2, R4, R5, R7, R8, R9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
