File: Hardware/ESP32_Thing_Plus.sch (EAGLE design)
At the start: 42 parts, among them Q1 2.5A/30V, Q2 MBT3904DW1T1, U1 MCP73831, U2 ESP-WROOM-32NARROW, U3 AP2112K-3.3V, U4 CP2102N

Commit message: v20
Added 10ohm series resistor between VUSB and CP2102
Parts:
- added R5: 10, SparkFun-Resistors:10OHM-0603-1/10W-5%
Connections:
- removed net 2: U2.IO2
- removed net 35: U2.IO35
- new net N$3: R5.2, U4.VBUS, U4.VREGIN
- net V_USB: now also R5.1; no longer U4.VBUS, U4.VREGIN
Other:
- note added: "v20"
- note removed: "v10"
- moved on the sheet: C19, C6, D1, JP2, R3, R6, U1
