File: Hardware/ESP32_Thing_Plus.brd (EAGLE design)
At the start: 22.9 x 58.4 mm, 107 parts, among them Q1 2.5A/30V, Q2 MBT3904DW1T1, U1 MCP73831, U2 ESP-WROOM-32NARROW, U3 AP2112K-3.3V, U4 CP2102N

Commit message: Updated USB to UART converter
Updated shematic to indicate the USB to UART converter can be either the CP2104 or CP2102N
Parts:
- U4: value CP2102N -> CP210X
Changed lines of the file:
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@@
 <attribute name="VALUE" x="1.778" y="11.049" size="0.6096" layer="27" font="vector" ratio="20" rot="R270"/>
 </element>
-<element name="U4" library="SparkFun-IC-Comms" package="QFN24" value="CP2102N" x="16.51" y="24.13" smashed="yes" rot="R90">
+<element name="U4" library="SparkFun-IC-Comms" package="QFN24" value="CP210X" x="16.51" y="24.13" smashed="yes" rot="R90">
 <attribute name="NAME" x="16.129" y="23.241" size="0.4064" layer="25" rot="R90"/>
 <attribute name="PROD_ID" value="IC-14020" x="16.51" y="24.13" size="1.778" layer="27" rot="R90" display="off"/>
